File: v2/redherring_v2.kicad_sch (KiCad schematic)
At the start: 187 parts, among them J4 Pimaroni Trackball, Q2 TIP120, SW1 SW_PUSH_LED, SW10 SW_PUSH_LED, SW11 SW_PUSH_LED, SW12 SW_PUSH_LED, SW13 SW_PUSH_LED, SW14 SW_PUSH_LED, SW15 SW_PUSH_LED, SW16 SW_PUSH_LED, SW17 SW_PUSH_LED, SW18 SW_PUSH_LED, SW19 SW_PUSH_LED, SW2 SW_PUSH_LED, SW20 SW_PUSH_LED, SW21 SW_PUSH_LED, SW22 SW_PUSH_LED, SW23 SW_PUSH_LED, SW24 SW_PUSH_LED, SW25 SW_PUSH_LED, SW26 SW_PUSH_LED, SW27 SW_PUSH_LED, SW28 SW_PUSH_LED, SW29 SW_PUSH_LED, SW3 SW_PUSH_LED, SW30 SW_PUSH_LED, SW31 SW_PUSH_LED, SW32 SW_PUSH_LED, SW33 SW_PUSH_LED, SW34 SW_PUSH_LED, SW35 SW_PUSH_LED, SW36 SW_PUSH_LED, SW37 SW_PUSH_LED, SW38 SW_PUSH_LED, SW39 SW_PUSH_LED, SW4 SW_PUSH_LED, SW40 SW_PUSH_LED, SW41 SW_PUSH_LED, SW42 SW_PUSH_LED, SW43 SW_PUSH_LED, SW44 SW_PUSH_LED, SW45 SW_PUSH_LED, SW46 SW_PUSH_LED, SW47 SW_PUSH_LED, SW48 SW_PUSH_LED, SW49 SW_PUSH_LED, SW5 SW_PUSH_LED, SW50 SW_PUSH_LED, SW51 SW_PUSH_LED, SW52 SW_PUSH_LED, SW53 SW_PUSH_LED, SW54 SW_PUSH_LED, SW55 SW_PUSH_LED, SW56 SW_PUSH_LED, SW57 SW_PUSH_LED, SW58 SW_PUSH_LED, SW59 SW_PUSH_LED, SW6 SW_PUSH_LED, SW60 SW_PUSH_LED, SW61 SW_PUSH_LED, SW62 SW_PUSH_LED, SW63 SW_PUSH_LED, SW64 SW_PUSH_LED, SW65 SW_PUSH_LED, SW66 SW_PUSH_LED, SW67 SW_PUSH_LED, SW68 SW_PUSH_LED, SW69 SW_PUSH_LED, SW7 SW_PUSH_LED, SW70 SW_PUSH_LED, SW71 SW_PUSH_LED, SW72 SW_PUSH_LED, SW73 SW_PUSH_LED, SW74 SW_PUSH_LED, SW75 SW_PUSH_LED, SW76 SW_PUSH_LED, SW77 SW_PUSH_LED, SW78 SW_PUSH_LED, SW79 SW_PUSH_LED, SW8 SW_PUSH_LED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

Commit message: Added level shifter Added decorative herringbone diodes
Parts:
- added D121: D, red_herring_v2_footprints:D_SOD-123_DO-35_Hybrid_DoubleSided, symbol Device:D
- added U2: SN74AHCT1G125, red_herring_v2_footprints:SN74AHCT1G125 - Junco, symbol Junco:SN74AHCT1G125
Connections:
- net GND: now also U2.1 (OE), U2.3 (GND)
- net LED: now also U2.2 (DIN); no longer SW7.4 (DIN)
- net VDD: no longer D_SOL_1.C, J4.1 (Pin_1), J_SOL_1.2 (Pin_2), SW1.1 (VDD), SW10.1 (VDD), SW11.1 (VDD), SW12.1 (VDD), SW13.1 (VDD), SW14.1 (VDD), SW15.1 (VDD), SW16.1 (VDD), SW17.1 (VDD), SW18.1 (VDD), SW19.1 (VDD), SW2.1 (VDD), SW20.1 (VDD), SW21.1 (VDD), SW22.1 (VDD), SW23.1 (VDD), SW24.1 (VDD), SW25.1 (VDD), SW26.1 (VDD), SW27.1 (VDD), SW28.1 (VDD), SW29.1 (VDD), SW3.1 (VDD), SW30.1 (VDD), SW31.1 (VDD), SW32.1 (VDD), SW33.1 (VDD), SW34.1 (VDD), SW35.1 (VDD), SW36.1 (VDD), SW37.1 (VDD), SW38.1 (VDD), SW39.1 (VDD), SW4.1 (VDD), SW40.1 (VDD), SW41.1 (VDD), SW42.1 (VDD), SW43.1 (VDD), SW44.1 (VDD), SW45.1 (VDD), SW46.1 (VDD), SW47.1 (VDD), SW48.1 (VDD), SW49.1 (VDD), SW5.1 (VDD), SW50.1 (VDD), SW51.1 (VDD), SW52.1 (VDD), SW53.1 (VDD), SW54.1 (VDD), SW55.1 (VDD), SW56.1 (VDD), SW57.1 (VDD), SW58.1 (VDD), SW59.1 (VDD), SW6.1 (VDD), SW60.1 (VDD), SW61.1 (VDD), SW62.1 (VDD), SW63.1 (VDD), SW64.1 (VDD), SW65.1 (VDD), SW66.1 (VDD), SW67.1 (VDD), SW68.1 (VDD), SW69.1 (VDD), SW7.1 (VDD), SW70.1 (VDD), SW71.1 (VDD), SW72.1 (VDD), SW73.1 (VDD), SW74.1 (VDD), SW75.1 (VDD), SW76.1 (VDD), SW77.1 (VDD), SW78.1 (VDD), SW79.1 (VDD), SW8.1 (VDD), SW80.1 (VDD), SW81.1 (VDD), SW82.1 (VDD), SW83.1 (VDD), SW84.1 (VDD), SW85.1 (VDD), SW86.1 (VDD), SW87.1 (VDD), SW88.1 (VDD), SW9.1 (VDD), U3.40 (VBUS)
- net VCC: now reaches U3.39 (VSYS)
- net VCC: now also D_SOL_1.C, J4.1 (Pin_1), J_SOL_1.2 (Pin_2), SW1.1 (VCC), SW10.1 (VCC), SW11.1 (VCC), SW12.1 (VCC), SW13.1 (VCC), SW14.1 (VCC), SW15.1 (VCC), SW16.1 (VCC), SW17.1 (VCC), SW18.1 (VCC), SW19.1 (VCC), SW2.1 (VCC), SW20.1 (VCC), SW21.1 (VCC), SW22.1 (VCC), SW23.1 (VCC), SW24.1 (VCC), SW25.1 (VCC), SW26.1 (VCC), SW27.1 (VCC), SW28.1 (VCC), SW29.1 (VCC), SW3.1 (VCC), SW30.1 (VCC), SW31.1 (VCC), SW32.1 (VCC), SW33.1 (VCC), SW34.1 (VCC), SW35.1 (VCC), SW36.1 (VCC), SW37.1 (VCC), SW38.1 (VCC), SW39.1 (VCC), SW4.1 (VCC), SW40.1 (VCC), SW41.1 (VCC), SW42.1 (VCC), SW43.1 (VCC), SW44.1 (VCC), SW45.1 (VCC), SW46.1 (VCC), SW47.1 (VCC), SW48.1 (VCC), SW49.1 (VCC), SW5.1 (VCC), SW50.1 (VCC), SW51.1 (VCC), SW52.1 (VCC), SW53.1 (VCC), SW54.1 (VCC), SW55.1 (VCC), SW56.1 (VCC), SW57.1 (VCC), SW58.1 (VCC), SW59.1 (VCC), SW6.1 (VCC), SW60.1 (VCC), SW61.1 (VCC), SW62.1 (VCC), SW63.1 (VCC), SW64.1 (VCC), SW65.1 (VCC), SW66.1 (VCC), SW67.1 (VCC), SW68.1 (VCC), SW69.1 (VCC), SW7.1 (VCC), SW70.1 (VCC), SW71.1 (VCC), SW72.1 (VCC), SW73.1 (VCC), SW74.1 (VCC), SW75.1 (VCC), SW76.1 (VCC), SW77.1 (VCC), SW78.1 (VCC), SW79.1 (VCC), SW8.1 (VCC), SW80.1 (VCC), SW81.1 (VCC), SW82.1 (VCC), SW83.1 (VCC), SW84.1 (VCC), SW85.1 (VCC), SW86.1 (VCC), SW87.1 (VCC), SW88.1 (VCC), SW9.1 (VCC), D121.1 (K), U2.5 (VCC)
- new net: D121.2 (A), U3.40 (VBUS)
- new net: SW7.4 (DIN), U2.4 (DOUT)
Other:
- note added: "LED Level shifter"
- note added: "The vbus/vsys and level shifter design were cribbed from the Junco: https://github.com/Daneski13/Junco#optional---rgb"

Commit message: Swqpped in updated OLED footprint Added pimaroni and updated footprint Started rerouting for pim and oled
Parts:
- J4: footprint red_herring_v2_footprints:pimoroni_trackball_tiein -> red_herring_v2_footprints:pimoroni_trackball
- OL1: footprint red_herring_v2_footprints:OLED 128x64 Double sided -> ergodonk_kicad_library:OLED SSD1306 128x64 UNVERIFIED
Changed lines of the file:
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@@
       (effects (font (size 1.1938 1.1938)) (justify left))
     )
-    (property "Footprint" "red_herring_v2_footprints:OLED 128x64 Double sided" (at 50.8 176.53 0)
+    (property "Footprint" "ergodonk_kicad_library:OLED SSD1306 128x64 UNVERIFIED" (at 50.8 176.53 0)
       (effects (font (size 1.524 1.524)) hide)
     )
@@
       (effects (font (size 1.27 1.27)) (justify left) hide)
     )
-    (property "Footprint" "red_herring_v2_footprints:pimoroni_trackball_tiein" (at 31.75 240.03 0)
+    (property "Footprint" "red_herring_v2_footprints:pimoroni_trackball" (at 31.75 240.03 0)
       (effects (font (size 1.27 1.27)) hide)
     )
